File: ThermalCam.kicad_pcb (KiCad board)
At the start: 2 copper layers, 44.9 x 47.2 mm, 100 parts, among them J1 Conn_02x20_Counter_Clockwise, J2 Conn_01x04, J3 Conn_01x06, Q1 BSS138PW,115, U1 GW1NR-9_QN882, U5 AP3012, U6 LT3042xMSE, U7 CAT24C128, U8 USBLC6-2SC6, U9 CY7C68013A-56PVX, X1 ASE-25MHz, Y1 24MHz

Commit message: Autoliv NV3 to UVC v1.0
Parts:
- added C31: 10u, Capacitor_SMD:C_0402_1005Metric, B.Cu at (152.3, 117.6)
- added C32: 10u, Capacitor_SMD:C_0402_1005Metric, B.Cu at (152.8, 109.8)
- added C33: 100n, Capacitor_SMD:C_0402_1005Metric, F.Cu at (146.6, 108.5)
- added C34: 100n, Capacitor_SMD:C_0402_1005Metric, F.Cu at (151.4, 110.7)
- added C35: 100n, Capacitor_SMD:C_0402_1005Metric, F.Cu at (164.8, 109.7)
- added C36: 100n, Capacitor_SMD:C_0402_1005Metric, F.Cu at (162.8, 103.5)
- added C37: 100n, Capacitor_SMD:C_0402_1005Metric, F.Cu at (164.2, 104.6)
- added C38: 100n, Capacitor_SMD:C_0402_1005Metric, F.Cu at (151.5, 104.9)
- added C39: 100n, Capacitor_SMD:C_0402_1005Metric, F.Cu at (152.3, 103.8)
- added C40: 100n, Capacitor_SMD:C_0402_1005Metric, F.Cu at (151.9, 115.2)
- added C41: 100n, Capacitor_SMD:C_0402_1005Metric, F.Cu at (154.2, 115.8)
- added C42: 100n, Capacitor_SMD:C_0402_1005Metric, F.Cu at (156.9, 115.8)
- added C43: 100n, Capacitor_SMD:C_0402_1005Metric, F.Cu at (164.2, 114.4)
- added C45: 100n, Capacitor_SMD:C_0402_1005Metric, F.Cu at (155.4, 99.9)
- added C46: 100n, Capacitor_SMD:C_0402_1005Metric, F.Cu at (158.8, 100.6)
- added C47: 100n, Capacitor_SMD:C_0402_1005Metric, F.Cu at (146.5, 90.4)
- added C48: 100n, Capacitor_SMD:C_0402_1005Metric, F.Cu at (165.8, 100.3)
- added C49: 100n, Capacitor_SMD:C_0402_1005Metric, F.Cu at (167.1, 87.8)
- added C50: 100n, Capacitor_SMD:C_0402_1005Metric, F.Cu at (164.9, 87.8)
- added C51: 100n, Capacitor_SMD:C_0402_1005Metric, F.Cu at (159.2, 87.8)
- added C52: 100n, Capacitor_SMD:C_0402_1005Metric, F.Cu at (154.4, 87.8)
- added C53: 100n, Capacitor_SMD:C_0402_1005Metric, F.Cu at (161.7, 87.8)
- added J4: USB_C_Receptacle, Connector_USB:USB_C_Receptacle_JAE_DX07S024WJ3R400, F.Cu at (149.8, 84.1)
- added U2: MUN3CAD01-SC, Custom:MUN3CAD01, F.Cu at (136.7, 88.4)
- added U3: MUN3CAD01-SC, Custom:MUN3CAD01, F.Cu at (132.7, 88.4)
- added U4: MUN3CAD01-SC, Custom:MUN3CAD01, F.Cu at (140.7, 88.4)
- added kibuzzard-636D73F4: G***, kibuzzard-636D73F4, F.Cu at (139.7, 80.5)
- added kibuzzard-636D7417: G***, kibuzzard-636D7417, F.Cu at (142.2, 102.1)
- added kibuzzard-636D7427: G***, kibuzzard-636D7427, F.Cu at (136.4, 102.1)
- added kibuzzard-636D7435: G***, kibuzzard-636D7435, F.Cu at (130.6, 102.1)
- added kibuzzard-636D765E: G***, kibuzzard-636D765E, B.Cu at (149.6, 102.4)
- C23, C24, C27: footprint Capacitor_SMD:C_0402_1005Metric -> Capacitor_SMD:C_0805_2012Metric
- C28: footprint Capacitor_SMD:C_0402_1005Metric -> Capacitor_SMD:C_0805_2012Metric; moved to B.Cu
- JP1, R1, R2, R8, R9: moved to B.Cu
- moved R30 99.8 mm to (148.1, 97.1), turned to 180 degrees
- moved R34 93.8 mm to (148.0, 88.5)
- moved R31 91.3 mm to (147.2, 80.6)
- moved JP2 88.9 mm to (145.2, 95.7), turned to 180 degrees
- moved U7 87.5 mm to (148.8, 92.8), turned to 90 degrees
- moved R33 86.7 mm to (151.0, 89.4), turned to 90 degrees
- moved R32 85.3 mm to (148.7, 87.6)
- moved FB6 82.3 mm to (141.8, 84.0), turned to 180 degrees
- moved C29 81.6 mm to (165.4, 85.4), turned to -90 degrees
- moved C21 80.4 mm to (137.1, 107.4), turned to 90 degrees
- moved Y1 79.7 mm to (163.2, 85.2), turned to -90 degrees
- moved R20 79.2 mm to (132.9, 90.7), turned to 180 degrees
- moved C7 78.0 mm to (137.1, 91.6), turned to 180 degrees
- moved C30 77.8 mm to (163.2, 82.7), turned to 180 degrees
- moved U8 77.0 mm to (158.3, 84.1), turned to 180 degrees
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Connections:
- net Net-(C10-Pad1) renamed /Power/2V5_UNFLT
- net Net-(C11-Pad1) renamed /Power/1V8_UNFLT
- net Net-(C12-Pad1) renamed /Power/3V3_UNFLT
- Q1 pad 1: V_{BIAS}_SEL -> /V_{BIAS}_SEL
- R26 pad 1: V_{BIAS}_SEL -> /V_{BIAS}_SEL
- U1 pad 17: /USB/FIFO_DATA0 -> /SHUTTER
- U1 pad 18: /USB/FIFO_DATA1 -> /USB/FIFO_CTRL.CLK_OUT
- U1 pad 19: /USB/FIFO_DATA2 -> /USB/FIFO_CTRL.SLRD
- U1 pad 20: /USB/FIFO_DATA3 -> /USB/FIFO_CTRL.SLWR
- U1 pad 25: /USB/FIFO_DATA4 -> /USB/FIFO_CTRL.CLK_IN
- U1 pad 26: /USB/FIFO_DATA5 -> /USB/FIFO_CTRL.PKTEND
- U1 pad 27: /USB/FIFO_DATA6 -> /USB/FIFO_CTRL.ADDR1
- U1 pad 28: /USB/FIFO_DATA7 -> /USB/FIFO_CTRL.ADDR0
- U1 pad 29: /USB/FIFO_CTRL.SLRD -> /USB/FIFO_CTRL.SLOE
- U1 pad 30: /USB/FIFO_CTRL.SLWR -> /USB/FIFO_CTRL.~{INT1}
- U1 pad 31: /USB/FIFO_CTRL.SLOE -> /USB/FIFO_CTRL.~{INT0}
- U1 pad 32: /USB/FIFO_CTRL.CLK_IN -> /USB/FIFO_CTRL.FLAG3
- U1 pad 33: /USB/FIFO_CTRL.CLK_OUT -> /USB/FIFO_CTRL.FLAG2
- U1 pad 35: /USB/FIFO_CTRL.FLAG2 -> /USB/FIFO_DATA7
- U1 pad 36: /USB/FIFO_CTRL.FLAG3 -> /USB/FIFO_DATA6
- U1 pad 37: /USB/FIFO_CTRL.~{INT0} -> /USB/FIFO_DATA5
- U1 pad 38: /USB/FIFO_CTRL.~{INT1} -> /USB/FIFO_DATA4
- U1 pad 39: /USB/FIFO_CTRL.ADDR0 -> /USB/FIFO_DATA0
- U1 pad 40: /USB/FIFO_CTRL.ADDR1 -> /USB/FIFO_DATA1
- U1 pad 41: /USB/FIFO_CTRL.PKTEND -> /USB/FIFO_DATA2
- U1 pad 42: /V_{BIAS}_SEL -> /USB/FIFO_DATA3
- U1 pad 47: /SHUTTER -> unconnected-(U1-Pad47)
- U1 pad 72: unconnected-(U1-Pad72) -> /V_{BIAS}_SEL
- U1 pad 89: (no net) -> GND
- U8 pad 2: /USB/V_{IN} -> +5V
Routing:
- net +3.3V: track 0.00 -> 52.2 mm, vias 0 -> 24
- net +2V5: track 0.00 -> 34.4 mm, vias 0 -> 2
- net /USB/FIFO_CTRL.CLK_IN: track 0.00 -> 32.8 mm
- net /FPGA_TMS: track 0.00 -> 28.2 mm
- net /FPGA_TCK: track 0.00 -> 26.7 mm
- net /USB/FIFO_CTRL.SLRD: track 0.00 -> 25.8 mm
- net /USB/FIFO_CTRL.CLK_OUT: track 0.00 -> 25.8 mm
- net /USB/FIFO_CTRL.SLWR: track 0.00 -> 25.3 mm
- net /FPGA_TDI: track 0.00 -> 25.2 mm
- net /FPGA_TDO: track 0.00 -> 24.6 mm
- net +5V: track 0.00 -> 23.2 mm, vias 0 -> 20
- net /USB/USB_D+: track 0.00 -> 21.9 mm, vias 0 -> 3
- net /USB/USB_D-: track 0.00 -> 21.4 mm, vias 0 -> 3
- net /USB/FIFO_DATA0: track 0.00 -> 18.6 mm
- net /USB/FIFO_DATA1: track 0.00 -> 18.4 mm
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- added copper zone on F.Cu, net +1V8
- added copper zone on In2.Cu, net +1V8
- added copper zone on F.Cu, net +3.3V
- added copper zone on In2.Cu, net +3.3V
- added copper zone on F.Cu, net +5V
- added copper zone on In2.Cu, net +5V
- added copper zone on B.Cu, net GND
- added copper zone on F.Cu, net GND
- added copper zone on In1.Cu, net GND
- added copper zone on F.Cu, net Net-(D13-Pad2)
Other:
- copper layers 2 -> 4
- board text added: "Autoliv NV3 to UVC v1.0"
- board text added: "JLCJLCJLCJLC"
- board text added: "by Dominik Sliwa dominik@sliwa.io"
- board text added: "dominik@sliwa.io"
