File: ThermalCam.kicad_sch (KiCad schematic)
At the start: 35 parts, among them J1 Conn_02x20_Counter_Clockwise, J2 Conn_01x04, J3 Conn_01x06, U1 GW1NR-9_QN882, X1 ASE-25MHz

Commit message: Autoliv NV3 to UVC v1.0
Parts:
- added C31, C32: 10u, Capacitor_SMD:C_0402_1005Metric, symbol Device:C_Small
- added C33, C34, C35, C36, C37, C38, C39, C40, C41, C42, C43: 100n, Capacitor_SMD:C_0402_1005Metric, symbol Device:C_Small
Connections:
- net +1V8: now also C35.1
- net +2V5: now also C32.1, C33.1, C34.1
- net +3.3V: now also C31.1, C36.1, C37.1, C38.1, C39.1, C40.1, C41.1, C42.1, C43.1
- net FIFO_CTRL.ADDR0: now also U1.28 (IOB11B); no longer U1.39 (IOB33A)
- net FIFO_CTRL.ADDR1: now also U1.27 (IOB11A); no longer U1.40 (IOB33B)
- net FIFO_CTRL.CLK_IN: now also U1.25 (IOB8A); no longer U1.32 (IOB15B)
- net FIFO_CTRL.CLK_OUT: now also U1.18 (IOB2B); no longer U1.33 (IOB23A)
- net FIFO_CTRL.FLAG2: now also U1.33 (IOB23A); no longer U1.35 (IOB29A/GCLKT_4)
- net FIFO_CTRL.FLAG3: now also U1.32 (IOB15B); no longer U1.36 (IOB29B/GCLKC_4)
- net FIFO_CTRL.PKTEND: now also U1.26 (IOB8B); no longer U1.41 (IOB41A)
- net FIFO_CTRL.SLOE: now also U1.29 (IOB13A); no longer U1.31 (IOB15A)
- net FIFO_CTRL.SLRD: now also U1.19 (IOB4A); no longer U1.29 (IOB13A)
- net FIFO_CTRL.SLWR: now also U1.20 (IOB4B); no longer U1.30 (IOB13B)
- net FIFO_CTRL.~{INT0}: now also U1.31 (IOB15A); no longer U1.37 (IOB31A)
- net FIFO_CTRL.~{INT1}: now also U1.30 (IOB13B); no longer U1.38 (IOB31B)
- net FIFO_DATA0: now also U1.39 (IOB33A); no longer U1.17 (IOB2A)
- net FIFO_DATA1: now also U1.40 (IOB33B); no longer U1.18 (IOB2B)
- net FIFO_DATA2: now also U1.41 (IOB41A); no longer U1.19 (IOB4A)
- net FIFO_DATA3: now also U1.42 (IOB41B); no longer U1.20 (IOB4B)
- net FIFO_DATA4: now also U1.38 (IOB31B); no longer U1.25 (IOB8A)
- net FIFO_DATA5: now also U1.37 (IOB31A); no longer U1.26 (IOB8B)
- net FIFO_DATA6: now also U1.36 (IOB29B/GCLKC_4); no longer U1.27 (IOB11A)
- net FIFO_DATA7: now also U1.35 (IOB29A/GCLKT_4); no longer U1.28 (IOB11B)
- net GND: now also U1.89 (VSS[6]), C31.2, C32.2, C33.2, C34.2, C35.2, C36.2, C37.2, C38.2, C39.2, C40.2, C41.2, C42.2, C43.2
- net SHUTTER: now also U1.17 (IOB2A); no longer U1.47 (IOB43B)
- net V_{BIAS}_SEL: now also U1.72 (IOT39B); no longer U1.42 (IOB41B)
- no-connect marks 21 -> 23
Other:
- sheet Power ports: added V_{BIAS}_SEL; removed none
