File: power.kicad_sch (KiCad schematic)
At the start: 53 parts, among them Q1 BSS138PW,115, U2 MUN3CAD01-SC, U3 MUN3CAD01-SC, U4 MUN3CAD01-SC, U5 AP3012, U6 LT3042xMSE

Commit message: Autoliv NV3 to UVC v1.0
Parts:
- C23, C24, C27, C28: footprint Capacitor_SMD:C_0402_1005Metric -> Capacitor_SMD:C_0805_2012Metric
- U2, U3, U4: footprint (none) -> Custom:MUN3CAD01
Connections:
- net 1V8_UNFLT: now reaches C11.1, C14.1, C8.1, FB2.1, R20.1, U3.6 (V_{OUT})
- net 2V5_UNFLT: now reaches C10.1, C13.1, C7.1, FB1.1, R18.1, U2.6 (V_{OUT})
- net 3V3_UNFLT: now reaches C12.1, C15.1, C9.1, FB3.1, R22.1, U4.6 (V_{OUT})
Changed lines of the file:
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@@
     (stroke (width 0) (type default) (color 0 0 0 0))
   )
-  (global_label "V_{BIAS}_SEL" (shape input) (at 196.342 62.738 180) (fields_autoplaced)
+  (label "3V3_UNFLT" (at 59.69 100.33 0)
+    (effects (font (size 1.27 1.27)) (justify left bottom))
+  )
+  (label "1V8_UNFLT" (at 56.388 23.622 0)
+    (effects (font (size 1.27 1.27)) (justify left bottom))
+  )
+  (label "2V5_UNFLT" (at 56.896 61.722 0)
+    (effects (font (size 1.27 1.27)) (justify left bottom))
+  )
+  (hierarchical_label "V_{BIAS}_SEL" (shape input) (at 196.342 62.738 180)
     (effects (font (size 1.27 1.27)) (justify right))
-    (property "Intersheet References" "${INTERSHEET_REFS}" (id 0) (at 185.1478 62.6586 0)
-      (effects (font (size 1.27 1.27)) (justify right) hide)
-    )
   )
   (symbol (lib_id "Device:R_Small") (at 60.706 35.052 0) (unit 1)
@@
       (effects (font (size 1.27 1.27)) (justify left))
     )
-    (property "Footprint" "Capacitor_SMD:C_0402_1005Metric" (id 2) (at 177.546 33.274 0)
+    (property "Footprint" "Capacitor_SMD:C_0805_2012Metric" (id 2) (at 177.546 33.274 0)
       (effects (font (size 1.27 1.27)) hide)
     )
@@
     (property "Reference" "U4" (id 0) (at 47.752 93.472 0))
     (property "Value" "MUN3CAD01-SC" (id 1) (at 47.752 96.012 0))
-    (property "Footprint" "" (id 2) (at 47.752 104.14 0)
+    (property "Footprint" "Custom:MUN3CAD01" (id 2) (at 47.752 104.14 0)
       (effects (font (size 1.27 1.27)) hide)
     )
@@
       (effects (font (size 1.27 1.27)) (justify left))
     )
-    (property "Footprint" "Capacitor_SMD:C_0402_1005Metric" (id 2) (at 189.484 33.02 0)
+    (property "Footprint" "Capacitor_SMD:C_0805_2012Metric" (id 2) (at 189.484 33.02 0)
       (effects (font (size 1.27 1.27)) hide)
     )
@@
       (effects (font (size 1.27 1.27)) (justify left))
     )
-    (property "Footprint" "Capacitor_SMD:C_0402_1005Metric" (id 2) (at 249.936 26.162 0)
+    (property "Footprint" "Capacitor_SMD:C_0805_2012Metric" (id 2) (at 249.936 26.162 0)
       (effects (font (size 1.27 1.27)) hide)
     )
@@
     (property "Reference" "U3" (id 0) (at 46.736 16.764 0))
     (property "Value" "MUN3CAD01-SC" (id 1) (at 46.736 19.304 0))
-    (property "Footprint" "" (id 2) (at 46.736 27.432 0)
+    (property "Footprint" "Custom:MUN3CAD01" (id 2) (at 46.736 27.432 0)
       (effects (font (size 1.27 1.27)) hide)
     )
@@
       (effects (font (size 1.27 1.27)) (justify left))
     )
-    (property "Footprint" "Capacitor_SMD:C_0402_1005Metric" (id 2) (at 261.112 26.416 0)
+    (property "Footprint" "Capacitor_SMD:C_0805_2012Metric" (id 2) (at 261.112 26.416 0)
       (effects (font (size 1.27 1.27)) hide)
     )
@@
     (property "Reference" "U2" (id 0) (at 46.482 54.864 0))
     (property "Value" "MUN3CAD01-SC" (id 1) (at 46.482 57.404 0))
-    (property "Footprint" "" (id 2) (at 46.482 65.532 0)
-      (effects (font (size 1.27 1.27)) hide)
-    )
+    (property "Footprint" "Custom:MUN3CAD01" (id 2) (at 46.482 65.532 0)
+      (effects (font (size 1.27 1.27)) hide)
+    )
