File: usb.kicad_sch (KiCad schematic)
At the start: 16 parts, among them J4 USB_C_Receptacle_USB2.0, U7 CAT24C128, U8 USBLC6-2SC6, U9 CY7C68013A-56PVX, Y1 24MHz

Commit message: Autoliv NV3 to UVC v1.0
Parts:
- removed J4: USB_C_Receptacle_USB2.0, symbol Connector:USB_C_Receptacle_USB2.0
- added C45, C46, C47, C48, C49, C50, C51, C52, C53: 100n, Capacitor_SMD:C_0402_1005Metric, symbol Device:C_Small
- added J4: USB_C_Receptacle, Connector_USB:USB_C_Receptacle_JAE_DX07S024WJ3R400, symbol Connector:USB_C_Receptacle
Connections:
- net +3.3V: now also C45.1, C46.1, C47.1, C48.1, C49.1, C50.1, C51.1, C52.1, C53.1
- net +5V: now also U8.2 (GND)
- net GND: now also C45.2, C46.2, C47.2, C48.2, C49.2, C50.2, C51.2, C52.2, C53.2, J4.A1 (GND), J4.A12 (GND), J4.B1 (GND), J4.B12 (GND), J4.S1 (SHIELD)
- net USB_D+: now also J4.A6 (D+), J4.B6 (D+)
- net USB_D-: now also J4.A7 (D-), J4.B7 (D-)
- net V_{IN}: now also J4.A4 (VBUS), J4.A9 (VBUS), J4.B4 (VBUS), J4.B9 (VBUS); no longer U8.2 (GND)
- net at R31.2: now also J4.A5 (CC1)
- net at R32.2: now also J4.B5 (CC2)
- no-connect marks 12 -> 20
Other:
- moved on the sheet: JP2, R30, U7
